File: Hardware/BlinkyCircuit.sch (EAGLE design)
At the start: 0 parts

Commit message: March 6 edits
Parts:
- added C1, C2, C4: (no value), LinnesLab-Passives:CAPACITOR0201
- added OP1, OP2: (no value), LinnesLab-AnalogIC:OP-DUALR
- added R1, R2, R3, R4: 10k, SparkFun-Resistors:10KOHM-0402-1/16W-1%
- added R5: (no value), LinnesLab-Passives:RESISTOR0201
- added R6: 13k, SparkFun-Resistors:13KOHM-0603-1/10W-1%
Connections:
- new net AGND: C2.2, OP2P.V-
- new net GND: C4.2, OP1P.V-, R2.1
- new net N$1: OP1B.+IN, R1.1, R2.2
- new net N$2: C1.1, OP1A.+IN, R5.1
- new net N$3: C1.2, OP1B.-IN, OP1B.OUT, R3.1
- new net N$4: OP1A.-IN, R3.2, R4.2
- new net N$5: OP1A.OUT, OP2B.-IN, R4.1, R5.2
- new net N$6: OP2B.+IN, OP2B.OUT
- new net V_BATT: C2.1, C4.1, OP1P.V+, OP2P.V+, R1.2
Other:
- note added: "Square Wave Generator"
