File: Hardware/BlinkyCircuit.sch (EAGLE design)
At the start: 11 parts

Commit message: March 13 2021 BlinkyCircuit schematic
Parts:
- added LED1, LED10, LED2, LED3, LED4, LED5, LED6, LED7, LED8, LED9: (no value), LinnesLab-LED:LED-4.SMD
- added Q1: (no value), LinnesLab-DiscreteSemi:NPN-GENERIC
Connections:
- new net N$7: Q1.B, R6.2
- new net N$8: LED1.C, LED10.C, LED2.C, LED3.C, LED4.C, LED5.C, LED6.C, LED7.C, LED8.C, LED9.C, Q1.C
- net AGND: now also Q1.E
- net N$6: now also R6.1
- net V_BATT: now also LED1.A, LED10.A, LED2.A, LED3.A, LED4.A, LED5.A, LED6.A, LED7.A, LED8.A, LED9.A
Other:
- moved on the sheet: R6

Commit message: March 22 2021 board edits
Parts:
- removed C1, C2, C4: (no value), LinnesLab-Passives:CAPACITOR0201
- removed LED10: (no value), LinnesLab-LED:LED-4.SMD
- removed R1, R2, R3, R4: 10k, SparkFun-Resistors:10KOHM-0402-1/16W-1%
- removed R5: (no value), LinnesLab-Passives:RESISTOR0201
- removed R6: 13k, SparkFun-Resistors:13KOHM-0603-1/10W-1%
- added C7, C8, C9: (no value), LinnesLab-Passives:CAPACITOR0603
- added LED21: (no value), LinnesLab-LED:LED5MM
- added R10, R11, R12, R7, R8, R9: (no value), LinnesLab-Passives:RESISTOR0603
- LED1, LED2, LED3, LED4, LED5, LED6, LED7, LED8, LED9: device LinnesLab-LED:LED-4.SMD -> LinnesLab-LED:LED5MM
Connections:
- removed net N$8: LED1.C, LED10.C, LED2.C, LED3.C, LED4.C, LED5.C, LED6.C, LED7.C, LED8.C, LED9.C, Q1.C
- new net N$11: LED1.C, LED2.C, LED21.C, LED3.C, LED4.C, LED5.C, LED6.C, LED7.C, LED8.C, LED9.C, Q1.C
- new net N$9: R7.2
- net AGND: now also C7.2; no longer C2.2, Q1.E
- net GND: now also C8.2, Q1.E, R9.1; no longer C4.2, R2.1
- net N$1: now also R7.1, R9.2; no longer R1.1, R2.2
- net N$2: now also C9.2, R8.1; no longer C1.1, R5.1
- net N$3: now also C9.1, R11.1; no longer C1.2, R3.1
- net N$4: now also R10.1, R11.2; no longer R3.2, R4.2
- net N$5: now also R10.2, R8.2; no longer R4.1, R5.2
- net N$6: now also R12.1; no longer R6.1
- net N$7: now also R12.2; no longer R6.2
- net V_BATT: now also C7.1, C8.1, LED21.A; no longer C2.1, C4.1, LED10.A, R1.2
Other:
- moved on the sheet: LED1, LED2, LED3, LED4, LED5, LED6, LED7

Commit message: March 22 2021 edits
Connections:
- net N$2: now also OP1A.-IN; no longer OP1A.+IN
- net N$4: now also OP1A.+IN; no longer OP1A.-IN
- net N$5: now also OP2B.+IN; no longer OP2B.-IN
- net N$6: now also OP2B.-IN; no longer OP2B.+IN
Other:
- moved on the sheet: OP1A, OP2B
Changed lines of the file:
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@@
 <attribute name="VALUE" x="19.05" y="35.56" size="1.778" layer="96"/>
 </instance>
-<instance part="OP1" gate="A" x="63.5" y="81.28" smashed="yes">
-<attribute name="NAME" x="66.04" y="84.455" size="1.778" layer="95"/>
-<attribute name="VALUE" x="66.04" y="76.2" size="1.778" layer="96"/>
+<instance part="OP1" gate="A" x="60.96" y="81.28" smashed="yes" rot="MR180">
+<attribute name="NAME" x="63.5" y="78.105" size="1.778" layer="95" rot="MR180"/>
+<attribute name="VALUE" x="63.5" y="86.36" size="1.778" layer="96" rot="MR180"/>
 </instance>
 <instance part="OP1" gate="B" x="17.78" y="40.64" smashed="yes">
@@
 <attribute name="VALUE" x="2.54" y="63.754" size="1.778" layer="96" align="bottom-center"/>
 </instance>
-<instance part="OP2" gate="B" x="109.22" y="78.74" smashed="yes">
-<attribute name="NAME" x="111.76" y="81.915" size="1.778" layer="95"/>
-<attribute name="VALUE" x="111.76" y="73.66" size="1.778" layer="96"/>
+<instance part="OP2" gate="B" x="109.22" y="78.74" smashed="yes" rot="MR180">
+<attribute name="NAME" x="111.76" y="75.565" size="1.778" layer="95" rot="MR180"/>
+<attribute name="VALUE" x="111.76" y="83.82" size="1.778" layer="96" rot="MR180"/>
 </instance>
 <instance part="SUPPLY3" gate="G$1" x="109.22" y="53.34" smashed="yes">
@@
 <net name="N$2" class="0">
 <segment>
-<pinref part="OP1" gate="A" pin="+IN"/>
 <wire x1="45.72" y1="83.82" x2="50.8" y2="83.82" width="0.1524" layer="91"/>
-<wire x1="50.8" y1="83.82" x2="55.88" y2="83.82" width="0.1524" layer="91"/>
 <wire x1="50.8" y1="93.98" x2="50.8" y2="83.82" width="0.1524" layer="91"/>
-<junction x="50.8" y="83.82"/>
 <wire x1="50.8" y1="93.98" x2="58.42" y2="93.98" width="0.1524" layer="91"/>
 <pinref part="R8" gate="G$1" pin="1"/>
 <pinref part="C9" gate="G$1" pin="2"/>
+<pinref part="OP1" gate="A" pin="-IN"/>
+<wire x1="50.8" y1="83.82" x2="53.34" y2="83.82" width="0.1524" layer="91"/>
+<junction x="50.8" y="83.82"/>
 </segment>
 </net>
 <net name="N$4" class="0">
 <segment>
-<pinref part="OP1" gate="A" pin="-IN"/>
-<wire x1="55.88" y1="78.74" x2="48.26" y2="78.74" width="0.1524" layer="91"/>
 <wire x1="48.26" y1="78.74" x2="48.26" y2="73.66" width="0.1524" layer="91"/>
 <wire x1="48.26" y1="73.66" x2="48.26" y2="71.12" width="0.1524" layer="91"/>
@@
 <pinref part="R10" gate="G$1" pin="1"/>
 <pinref part="R11" gate="G$1" pin="2"/>
+<pinref part="OP1" gate="A" pin="+IN"/>
+<wire x1="53.34" y1="78.74" x2="48.26" y2="78.74" width="0.1524" layer="91"/>
 </segment>
 </net>
@@
 <wire x1="68.58" y1="93.98" x2="78.74" y2="93.98" width="0.1524" layer="91"/>
 <wire x1="78.74" y1="93.98" x2="78.74" y2="81.28" width="0.1524" layer="91"/>
+<wire x1="78.74" y1="81.28" x2="78.74" y2="76.2" width="0.1524" layer="91"/>
+<wire x1="78.74" y1="76.2" x2="78.74" y2="73.66" width="0.1524" layer="91"/>
+<wire x1="71.12" y1="73.66" x2="78.74" y2="73.66" width="0.1524" layer="91"/>
+<pinref part="R8" gate="G$1" pin="2"/>
+<pinref part="R10" gate="G$1" pin="2"/>
 <pinref part="OP1" gate="A" pin="OUT"/>
-<wire x1="78.74" y1="81.28" x2="71.12" y2="81.28" width="0.1524" layer="91"/>
-<wire x1="71.12" y1="73.66" x2="78.74" y2="73.66" width="0.1524" layer="91"/>
-<wire x1="78.74" y1="73.66" x2="78.74" y2="76.2" width="0.1524" layer="91"/>
+<wire x1="68.58" y1="81.28" x2="78.74" y2="81.28" width="0.1524" layer="91"/>
 <junction x="78.74" y="81.28"/>
-<pinref part="OP2" gate="B" pin="-IN"/>
-<wire x1="78.74" y1="76.2" x2="78.74" y2="81.28" width="0.1524" layer="91"/>
+<pinref part="OP2" gate="B" pin="+IN"/>
 <wire x1="101.6" y1="76.2" x2="78.74" y2="76.2" width="0.1524" layer="91"/>
 <junction x="78.74" y="76.2"/>
-<pinref part="R8" gate="G$1" pin="2"/>
-<pinref part="R10" gate="G$1" pin="2"/>
 </segment>
 </net>
 <net name="N$6" class="0">
 <segment>
-<pinref part="OP2" gate="B" pin="+IN"/>
-<wire x1="101.6" y1="81.28" x2="96.52" y2="81.28" width="0.1524" layer="91"/>
 <wire x1="96.52" y1="81.28" x2="96.52" y2="88.9" width="0.1524" layer="91"/>
 <wire x1="96.52" y1="88.9" x2="124.46" y2="88.9" width="0.1524" layer="91"/>
 <wire x1="124.46" y1="88.9" x2="124.46" y2="78.74" width="0.1524" layer="91"/>
+<wire x1="124.46" y1="78.74" x2="129.54" y2="78.74" width="0.1524" layer="91"/>
+<pinref part="R12" gate="G$1" pin="1"/>
+<pinref part="OP2" gate="B" pin="-IN"/>
+<wire x1="96.52" y1="81.28" x2="101.6" y2="81.28" width="0.1524" layer="91"/>
 <pinref part="OP2" gate="B" pin="OUT"/>
-<wire x1="124.46" y1="78.74" x2="116.84" y2="78.74" width="0.1524" layer="91"/>
-<wire x1="124.46" y1="78.74" x2="129.54" y2="78.74" width="0.1524" layer="91"/>
+<wire x1="116.84" y1="78.74" x2="124.46" y2="78.74" width="0.1524" layer="91"/>
 <junction x="124.46" y="78.74"/>
-<pinref part="R12" gate="G$1" pin="1"/>
-</segment>
-</net>
+</segment>
+</net>

Commit message: March 22 2021 edits
Connections:
- removed net N$9: R7.2
- net V_BATT: now also R7.2
Changed lines of the file:
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@@
 <net name="V_BATT" class="0">
-<segment>
-<pinref part="SUPPLY2" gate="G$1" pin="V_BATT"/>
-<wire x1="2.54" y1="60.96" x2="2.54" y2="55.88" width="0.1524" layer="91"/>
-</segment>
 <segment>
 <pinref part="SUPPLY1" gate="G$1" pin="V_BATT"/>
@@
 <wire x1="180.34" y1="93.98" x2="185.42" y2="93.98" width="0.1524" layer="91"/>
 <junction x="180.34" y="93.98"/>
+</segment>
+<segment>
+<pinref part="R7" gate="G$1" pin="2"/>
+<pinref part="SUPPLY2" gate="G$1" pin="V_BATT"/>
+<wire x1="2.54" y1="55.88" x2="2.54" y2="60.96" width="0.1524" layer="91"/>
 </segment>
 </net>
@@
 </segment>
 </net>
-<net name="N$9" class="0">
-<segment>
-<pinref part="R7" gate="G$1" pin="2"/>
-<junction x="2.54" y="55.88"/>
-</segment>
-</net>

Commit message: March 222 2021 edits
Connections:
- removed net AGND: C7.2, OP2P.V-
- net GND: now also C7.2, OP2P.V-
Changed lines of the file:
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@@
 <part name="OP2" library="LinnesLab-AnalogIC" deviceset="OP-DUAL" device="R" package3d_urn="urn:adsk.eagle:package:15818288/2"/>
 <part name="SUPPLY3" library="LinnesLab-Symbols" deviceset="VBATT" device=""/>
-<part name="AGND1" library="LinnesLab-Symbols" deviceset="AGND" device=""/>
 <part name="SUPPLY5" library="LinnesLab-Symbols" deviceset="VBATT" device=""/>
 <part name="Q1" library="LinnesLab-DiscreteSemi" deviceset="NPN" device="-GENERIC" package3d_urn="urn:adsk.eagle:package:15662047/2"/>
@@
 <attribute name="VALUE" x="109.22" y="56.134" size="1.778" layer="96" align="bottom-center"/>
 </instance>
-<instance part="AGND1" gate="G$1" x="109.22" y="25.4" smashed="yes">
-<attribute name="VALUE" x="109.22" y="22.606" size="1.778" layer="96" align="top-center"/>
-</instance>
 <instance part="OP2" gate="P" x="109.22" y="40.64" smashed="yes">
 <attribute name="NAME" x="110.49" y="44.45" size="1.778" layer="95"/>
@@
 <pinref part="Q1" gate="G$1" pin="E"/>
 <wire x1="149.86" y1="73.66" x2="149.86" y2="12.7" width="0.1524" layer="91"/>
-<wire x1="149.86" y1="12.7" x2="66.04" y2="12.7" width="0.1524" layer="91"/>
+<wire x1="149.86" y1="12.7" x2="109.22" y2="12.7" width="0.1524" layer="91"/>
+<pinref part="OP2" gate="P" pin="V-"/>
+<wire x1="109.22" y1="12.7" x2="66.04" y2="12.7" width="0.1524" layer="91"/>
+<wire x1="109.22" y1="33.02" x2="109.22" y2="27.94" width="0.1524" layer="91"/>
+<wire x1="109.22" y1="27.94" x2="101.6" y2="27.94" width="0.1524" layer="91"/>
+<wire x1="101.6" y1="27.94" x2="101.6" y2="35.56" width="0.1524" layer="91"/>
+<pinref part="C7" gate="G$1" pin="2"/>
+<wire x1="109.22" y1="27.94" x2="109.22" y2="12.7" width="0.1524" layer="91"/>
+<junction x="109.22" y="27.94"/>
+<junction x="109.22" y="12.7"/>
 </segment>
 </net>
@@
 </segment>
 </net>
-<net name="AGND" class="0">
-<segment>
-<pinref part="OP2" gate="P" pin="V-"/>
-<pinref part="AGND1" gate="G$1" pin="AGND"/>
-<wire x1="109.22" y1="33.02" x2="109.22" y2="27.94" width="0.1524" layer="91"/>
-<wire x1="109.22" y1="27.94" x2="101.6" y2="27.94" width="0.1524" layer="91"/>
-<junction x="109.22" y="27.94"/>
-<wire x1="101.6" y1="27.94" x2="101.6" y2="35.56" width="0.1524" layer="91"/>
-<pinref part="C7" gate="G$1" pin="2"/>
-</segment>
-</net>

Commit message: March 27 2021 edits
Parts:
- added J1: (no value), LinnesLab-Connectors:CONN_02
Connections:
- net GND: now also J1.2
- net V_BATT: now also J1.1
Changed lines of the file:
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@@
 <part name="LED9" library="LinnesLab-LED" deviceset="LED" device="5MM"/>
 <part name="GND4" library="LinnesLab-Symbols" deviceset="GND" device=""/>
+<part name="J1" library="LinnesLab-Connectors" deviceset="CONN_02" device=""/>
 </parts>
 <sheets>
@@
 <attribute name="VALUE" x="66.04" y="9.906" size="1.778" layer="96" align="top-center"/>
 </instance>
+<instance part="J1" gate="G$1" x="17.78" y="68.58" smashed="yes" rot="R270">
+<attribute name="VALUE" x="12.954" y="71.12" size="1.778" layer="96" font="vector" rot="R270"/>
+<attribute name="NAME" x="23.368" y="71.12" size="1.778" layer="95" font="vector" rot="R270"/>
+</instance>
 </instances>
 <busses>
@@
 <wire x1="2.54" y1="12.7" x2="17.78" y2="12.7" width="0.1524" layer="91"/>
 <pinref part="OP1" gate="P" pin="V-"/>
-<wire x1="17.78" y1="12.7" x2="66.04" y2="12.7" width="0.1524" layer="91"/>
+<wire x1="17.78" y1="12.7" x2="20.32" y2="12.7" width="0.1524" layer="91"/>
+<wire x1="22.86" y1="12.7" x2="66.04" y2="12.7" width="0.1524" layer="91"/>
 <wire x1="17.78" y1="33.02" x2="17.78" y2="12.7" width="0.1524" layer="91"/>
 <pinref part="C8" gate="G$1" pin="2"/>
@@
 <junction x="109.22" y="27.94"/>
 <junction x="109.22" y="12.7"/>
+<pinref part="J1" gate="G$1" pin="2"/>
+<wire x1="20.32" y1="60.96" x2="20.32" y2="12.7" width="0.1524" layer="91"/>
+<wire x1="20.32" y1="12.7" x2="22.86" y2="12.7" width="0.1524" layer="91"/>
 </segment>
 </net>
@@
 <junction x="17.78" y="50.8"/>
 <pinref part="C8" gate="G$1" pin="1"/>
+<pinref part="J1" gate="G$1" pin="1"/>
+<wire x1="17.78" y1="60.96" x2="17.78" y2="53.34" width="0.1524" layer="91"/>
+<junction x="17.78" y="53.34"/>
 </segment>
 <segment>
