File: Hardware/BlinkyCircuit.brd (EAGLE design)
At the start: 160 x 100 mm, 0 parts

Commit message: March 6 edits
Parts:
- added C1, C2, C4: (no value), LinnesLab-Passives:C0201
- added OP1, OP2: (no value), LinnesLab-AnalogIC:SO8
- added R1, R2, R3, R4: 10k, SparkFun-Resistors:0402
- added R5: (no value), LinnesLab-Passives:R0201
- added R6: 13k, SparkFun-Resistors:0603
Connections:
- new net AGND: C2.2, OP2.4
- new net GND: C4.2, OP1.4, R2.1
- new net N$1: OP1.5, R1.1, R2.2
- new net N$2: C1.1, OP1.3, R5.1
- new net N$3: C1.2, OP1.6, OP1.7, R3.1
- new net N$4: OP1.2, R3.2, R4.2
- new net N$5: OP1.1, OP2.6, R4.1, R5.2
- new net N$6: OP2.5, OP2.7
- new net V_BATT: C2.1, C4.1, OP1.8, OP2.8, R1.2

Commit message: March 13 2021 BlinkyCircuit schematic
Parts:
- added LED1, LED10, LED2, LED3, LED4, LED5, LED6, LED7, LED8, LED9: (no value), LinnesLab-LED:4-SMD
- added Q1: (no value), LinnesLab-DiscreteSemi:SOT23-3
Connections:
- new net N$7: Q1.1, R6.2
- new net N$8: LED1.2.1, LED1.2.2, LED10.2.1, LED10.2.2, LED2.2.1, LED2.2.2, LED3.2.1, LED3.2.2, LED4.2.1, LED4.2.2, LED5.2.1, LED5.2.2, LED6.2.1, LED6.2.2, LED7.2.1, LED7.2.2, LED8.2.1, LED8.2.2, LED9.2.1, LED9.2.2, Q1.3
- net AGND: now also Q1.2
- net N$6: now also R6.1
- net V_BATT: now also LED1.1.1, LED1.1.2, LED10.1.1, LED10.1.2, LED2.1.1, LED2.1.2, LED3.1.1, LED3.1.2, LED4.1.1, LED4.1.2, LED5.1.1, LED5.1.2, LED6.1.1, LED6.1.2, LED7.1.1, LED7.1.2, LED8.1.1, LED8.1.2, LED9.1.1, LED9.1.2

Commit message: March 13 2021 board edits
Parts:
- moved OP1 158.5 mm to (124.5, 14.0)
- moved R1 24.4 mm to (14.0, 3.81)
- moved LED6 22.5 mm to (6.35, -127.0)
- moved LED7 22.5 mm to (6.35, -133.3)
- moved LED8 22.5 mm to (6.35, -139.7)
- moved LED3 22.5 mm to (6.35, -108.0)
- moved LED4 22.5 mm to (6.35, -114.3)
- moved LED10 22.5 mm to (6.35, -152.4)
- moved LED5 22.5 mm to (6.35, -120.7)
- moved LED9 22.5 mm to (6.35, -146.1)
- moved R2 6.48 mm to (-3.81, -8.89)
Other:
- board size 160 x 100 mm -> 152.4 x 152.4 mm

Commit message: March 22 2021 board edits
Parts:
- removed C1, C2, C4: (no value), LinnesLab-Passives:C0201
- removed LED10: (no value), LinnesLab-LED:4-SMD
- removed R1, R2, R3, R4: 10k, SparkFun-Resistors:0402
- removed R5: (no value), LinnesLab-Passives:R0201
- removed R6: 13k, SparkFun-Resistors:0603
- added C7, C8, C9: (no value), LinnesLab-Passives:C0603
- added LED21: (no value), LinnesLab-LED:LED_5MM
- added R10, R11, R12, R7, R8, R9: (no value), LinnesLab-Passives:R0603
- LED1, LED2, LED3, LED4, LED5, LED6, LED7, LED8, LED9: device LinnesLab-LED:4-SMD -> LinnesLab-LED:LED_5MM
- moved LED1 185.1 mm to (-80.0, -275.6)
- moved LED9 170.8 mm to (-80.0, -293.4)
- moved LED8 168.6 mm to (-80.0, -284.5)
- moved LED7 151.5 mm to (-80.0, -257.8)
- moved LED6 149.4 mm to (-80.0, -248.9)
- moved LED5 147.3 mm to (-80.0, -240.0)
- moved LED4 145.3 mm to (-80.0, -231.1)
- moved LED3 143.3 mm to (-80.0, -222.2)
- moved LED2 119.1 mm to (-80.0, -213.4)
Connections:
- removed net N$8: LED1.2.1, LED1.2.2, LED10.2.1, LED10.2.2, LED2.2.1, LED2.2.2, LED3.2.1, LED3.2.2, LED4.2.1, LED4.2.2, LED5.2.1, LED5.2.2, LED6.2.1, LED6.2.2, LED7.2.1, LED7.2.2, LED8.2.1, LED8.2.2, LED9.2.1, LED9.2.2, Q1.3
- new net N$11: LED1.K, LED2.K, LED21.K, LED3.K, LED4.K, LED5.K, LED6.K, LED7.K, LED8.K, LED9.K, Q1.3
- new net N$9: R7.2
- net AGND: now also C7.2; no longer C2.2, Q1.2
- net GND: now also C8.2, Q1.2, R9.1; no longer C4.2, R2.1
- net N$1: now also R7.1, R9.2; no longer R1.1, R2.2
- net N$2: now also C9.2, R8.1; no longer C1.1, R5.1
- net N$3: now also C9.1, R11.1; no longer C1.2, R3.1
- net N$4: now also R10.1, R11.2; no longer R3.2, R4.2
- net N$5: now also R10.2, R8.2; no longer R4.1, R5.2
- net N$6: now also R12.1; no longer R6.1
- net N$7: now also R12.2; no longer R6.2
- net V_BATT: now also C7.1, C8.1, LED1.A, LED2.A, LED21.A, LED3.A, LED4.A, LED5.A, LED6.A, LED7.A, LED8.A, LED9.A; no longer C2.1, C4.1, LED1.1.1, LED1.1.2, LED10.1.1, LED10.1.2, LED2.1.1, LED2.1.2, LED3.1.1, LED3.1.2, LED4.1.1, LED4.1.2, LED5.1.1, LED5.1.2, LED6.1.1, LED6.1.2, LED7.1.1, LED7.1.2, LED8.1.1, LED8.1.2, LED9.1.1, LED9.1.2, R1.2

Commit message: March 22 2021 edits
Connections:
- net N$2: now also OP1.2; no longer OP1.3
- net N$4: now also OP1.3; no longer OP1.2
- net N$5: now also OP2.5; no longer OP2.6
- net N$6: now also OP2.6; no longer OP2.5
Changed lines of the file:
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@@
 <setting verticaltext="up"/>
 </settings>
-<grid distance="50" unitdist="mil" unit="mil" style="lines" multiple="1" display="no" altdistance="5" altunitdist="mil" altunit="mil"/>
+<grid distance="100" unitdist="mil" unit="mil" style="lines" multiple="1" display="no" altdistance="5" altunitdist="mil" altunit="mil"/>
 <layers>
 <layer number="1" name="Top" color="4" fill="1" visible="yes" active="yes"/>
@@
 </signal>
 <signal name="N$2">
-<contactref element="OP1" pad="3"/>
 <contactref element="R8" pad="1"/>
 <contactref element="C9" pad="2"/>
+<contactref element="OP1" pad="2"/>
 <wire x1="-12.28" y1="-160.02" x2="-10.58" y2="-198.12" width="0" layer="19" extent="1-1"/>
-<wire x1="125.095" y1="11.37" x2="-12.28" y2="-160.02" width="0" layer="19" extent="1-1"/>
+<wire x1="123.825" y1="11.37" x2="-12.28" y2="-160.02" width="0" layer="19" extent="1-1"/>
 </signal>
 <signal name="N$4">
-<contactref element="OP1" pad="2"/>
 <contactref element="R10" pad="1"/>
 <contactref element="R11" pad="2"/>
+<contactref element="OP1" pad="3"/>
 <wire x1="-12.28" y1="-167.64" x2="-10.58" y2="-171.45" width="0" layer="19" extent="1-1"/>
-<wire x1="123.825" y1="11.37" x2="-12.28" y2="-167.64" width="0" layer="19" extent="1-1"/>
+<wire x1="125.095" y1="11.37" x2="-12.28" y2="-167.64" width="0" layer="19" extent="1-1"/>
 </signal>
 <signal name="N$5">
-<contactref element="OP1" pad="1"/>
-<contactref element="OP2" pad="6"/>
 <contactref element="R8" pad="2"/>
 <contactref element="R10" pad="2"/>
+<contactref element="OP1" pad="1"/>
+<contactref element="OP2" pad="5"/>
 <wire x1="-10.58" y1="-160.02" x2="-10.58" y2="-167.64" width="0" layer="19" extent="1-1"/>
-<wire x1="-0.635" y1="-93.92" x2="-10.58" y2="-160.02" width="0" layer="19" extent="1-1"/>
-<wire x1="122.555" y1="11.37" x2="-0.635" y2="-93.92" width="0" layer="19" extent="1-1"/>
+<wire x1="0.635" y1="-93.92" x2="-10.58" y2="-160.02" width="0" layer="19" extent="1-1"/>
+<wire x1="122.555" y1="11.37" x2="0.635" y2="-93.92" width="0" layer="19" extent="1-1"/>
 </signal>
 <signal name="N$6">
-<contactref element="OP2" pad="5"/>
+<contactref element="R12" pad="1"/>
+<contactref element="OP2" pad="6"/>
 <contactref element="OP2" pad="7"/>
-<contactref element="R12" pad="1"/>
 <wire x1="-1.905" y1="-93.92" x2="-12.28" y2="-175.26" width="0" layer="19" extent="1-1"/>
-<wire x1="0.635" y1="-93.92" x2="-1.905" y2="-93.92" width="0" layer="19" extent="1-1"/>
+<wire x1="-0.635" y1="-93.92" x2="-1.905" y2="-93.92" width="0" layer="19" extent="1-1"/>
 </signal>
 <signal name="AGND">

Commit message: March 22 2021 edits
Parts:
- moved LED2 178.5 mm to (-34.8, -40.7)
- moved LED3 172.3 mm to (-34.8, -56.0)
- moved LED4 169.5 mm to (-35.5, -67.6)
- moved LED5 164.6 mm to (-34.5, -81.9)
- moved LED6 159.0 mm to (-32.5, -97.2)
- moved LED7 155.5 mm to (-27.4, -111.5)
- moved LED21 149.9 mm to (-26.0, -126.8)
- moved LED1 147.3 mm to (-25.5, -138.7)
- moved LED8 145.2 mm to (-23.9, -150.6)
- moved LED9 141.8 mm to (-23.2, -163.5)
- moved OP1 115.9 mm to (8.59, 16.9)
- moved C7 109.2 mm to (9.75, -83.4)
- moved C8 109.2 mm to (9.75, -87.2)
- moved C9 109.2 mm to (9.75, -91.0)
- moved R7 109.2 mm to (9.75, -49.1)
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Connections:
- removed net N$9: R7.2
- net V_BATT: now also R7.2
Other:
- board size 152.4 x 152.4 mm -> 25.4 x 25.4 mm

Commit message: March 222 2021 edits
Parts:
- moved LED9 132.9 mm to (-18.4, -30.7)
- moved LED8 129.0 mm to (-18.0, -21.8)
- moved LED1 125.9 mm to (-14.9, -13.2)
- moved LED21 119.0 mm to (-10.1, -8.89)
- moved LED7 107.1 mm to (-6.48, -6.40)
- moved LED6 94.7 mm to (1.98, -8.92)
- moved C7 87.3 mm to (38.3, -0.84)
- moved LED5 86.1 mm to (4.06, -4.95)
- moved C9 84.1 mm to (8.99, -6.91)
- moved C8 80.5 mm to (17.3, -7.06)
- moved LED4 77.5 mm to (2.46, -0.10)
- moved LED3 72.9 mm to (2.54, 6.53)
- moved LED2 65.8 mm to (2.67, 13.4)
- moved R12 60.2 mm to (19.0, -8.66)
- moved R9 59.7 mm to (16.4, 2.67)
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Connections:
- removed net AGND: C7.2, OP2.4
- net GND: now also C7.2, OP2.4

Commit message: March 22 2021 board edits
Other:
- board size 25.4 x 25.4 mm -> 170.5 x 81 mm
Changed lines of the file:
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@@
 <board>
 <plain>
-<dimension x1="160" y1="100" x2="0" y2="100" x3="80" y3="110.49" textsize="1.778" layer="1"/>
-<wire x1="0" y1="0" x2="25.4" y2="0" width="0.1524" layer="20"/>
-<wire x1="25.4" y1="0" x2="25.4" y2="25.4" width="0.1524" layer="20"/>
-<wire x1="25.4" y1="25.4" x2="0" y2="25.4" width="0.1524" layer="20"/>
-<wire x1="0" y1="25.4" x2="0" y2="0" width="0.1524" layer="20"/>
+<wire x1="110.7948" y1="109.474" x2="120.4722" y2="119.1006" width="0.1524" layer="20" curve="-90"/>
+<wire x1="120.4722" y1="119.1006" x2="128.6002" y2="119.1006" width="0.1524" layer="20"/>
+<wire x1="128.6002" y1="119.1006" x2="136.7282" y2="110.9726" width="0.1524" layer="20" curve="-90"/>
+<wire x1="136.7282" y1="110.9726" x2="136.9822" y2="107.3658" width="0.1524" layer="20"/>
+<wire x1="136.9822" y1="107.3658" x2="148.0566" y2="118.6942" width="0.1524" layer="20" curve="-90"/>
+<wire x1="148.0566" y1="118.6942" x2="155.3718" y2="118.6942" width="0.1524" layer="20"/>
+<wire x1="155.3718" y1="118.6942" x2="165.9382" y2="108.1278" width="0.1524" layer="20" curve="-90"/>
+<wire x1="165.9382" y1="108.1278" x2="165.9382" y2="104.9274" width="0.1524" layer="20"/>
+<wire x1="165.9382" y1="104.9274" x2="169.5958" y2="108.585" width="0.1524" layer="20" curve="-90"/>
+<wire x1="169.5958" y1="108.585" x2="215.011" y2="108.585" width="0.1524" layer="20"/>
+<wire x1="215.011" y1="108.585" x2="217.8558" y2="105.7402" width="0.1524" layer="20" curve="-90"/>
+<wire x1="217.8558" y1="105.7402" x2="217.8558" y2="104.9274" width="0.1524" layer="20"/>
+<wire x1="217.8558" y1="104.9274" x2="223.52" y2="110.5916" width="0.1524" layer="20" curve="-90"/>
+<wire x1="223.52" y1="110.5916" x2="232.8672" y2="110.5916" width="0.1524" layer="20"/>
+<wire x1="232.8672" y1="110.5916" x2="238.9632" y2="104.4956" width="0.1524" layer="20" curve="-90"/>
+<wire x1="238.9632" y1="104.4956" x2="238.9632" y2="96.012" width="0.1524" layer="20"/>
+<wire x1="238.9632" y1="96.012" x2="206.9592" y2="64.008" width="0.1524" layer="20" curve="-90"/>
+<wire x1="206.9592" y1="64.008" x2="193.5226" y2="64.008" width="0.1524" layer="20"/>
+<wire x1="110.7948" y1="109.474" x2="68.5038" y2="67.183" width="0.1524" layer="20" curve="90"/>
+<wire x1="68.5038" y1="67.183" x2="68.5038" y2="66.0908" width="0.1524" layer="20"/>
+<wire x1="68.6308" y1="66.3194" x2="96.774" y2="38.1762" width="0.1524" layer="20" curve="90"/>
+<wire x1="96.774" y1="38.1762" x2="157.1244" y2="38.1" width="0.1524" layer="20"/>
+<wire x1="193.5226" y1="64.008" x2="157.1244" y2="38.1" width="0.1524" layer="20"/>
 </plain>
 <attributes>
@@
 <contactref element="R7" pad="1"/>
 <contactref element="R9" pad="2"/>
+<wire x1="17.2838" y1="2.667" x2="10.4902" y2="24.2154" width="0" layer="19" extent="1-1"/>
 <wire x1="19.0128" y1="2.5654" x2="17.2838" y2="2.667" width="0" layer="19" extent="1-1"/>
-<wire x1="10.4902" y1="24.2154" x2="19.0128" y2="2.5654" width="0" layer="19" extent="1-1"/>
 </signal>
 <signal name="GND">
@@
 <wire x1="1.27" y1="6.5278" x2="1.1938" y2="-0.1016" width="0" layer="19" extent="1-1"/>
 <wire x1="1.397" y1="13.3604" x2="1.27" y2="6.5278" width="0" layer="19" extent="1-1"/>
-<wire x1="16.4728" y1="-7.0612" x2="0.7112" y2="-8.9154" width="0" layer="19" extent="1-1"/>
-<wire x1="37.4024" y1="-0.8382" x2="16.4728" y2="-7.0612" width="0" layer="19" extent="1-1"/>
-<wire x1="20.7128" y1="2.5654" x2="37.4024" y2="-0.8382" width="0" layer="19" extent="1-1"/>
-<wire x1="17.6784" y1="22.9962" x2="20.7128" y2="2.5654" width="0" layer="19" extent="1-1"/>
-<wire x1="6.6802" y1="24.2154" x2="17.6784" y2="22.9962" width="0" layer="19" extent="1-1"/>
+<wire x1="6.6802" y1="24.2154" x2="1.397" y2="13.3604" width="0" layer="19" extent="1-1"/>
+<wire x1="17.6784" y1="22.9962" x2="6.6802" y2="24.2154" width="0" layer="19" extent="1-1"/>
+<wire x1="16.4728" y1="-7.0612" x2="2.794" y2="-4.953" width="0" layer="19" extent="1-1"/>
+<wire x1="20.7128" y1="2.5654" x2="16.4728" y2="-7.0612" width="0" layer="19" extent="1-1"/>
+<wire x1="37.4024" y1="-0.8382" x2="20.7128" y2="2.5654" width="0" layer="19" extent="1-1"/>
 </signal>
 <signal name="N$3">
@@
 <contactref element="R11" pad="1"/>
 <contactref element="C9" pad="1"/>
+<wire x1="7.9502" y1="24.2154" x2="9.2202" y2="24.2154" width="0" layer="19" extent="1-1"/>
+<wire x1="8.1416" y1="-6.9088" x2="7.9502" y2="24.2154" width="0" layer="19" extent="1-1"/>
 <wire x1="10.2498" y1="-9.525" x2="8.1416" y2="-6.9088" width="0" layer="19" extent="1-1"/>
-<wire x1="9.2202" y1="24.2154" x2="10.2498" y2="-9.525" width="0" layer="19" extent="1-1"/>
-<wire x1="7.9502" y1="24.2154" x2="9.2202" y2="24.2154" width="0" layer="19" extent="1-1"/>
 </signal>
 <signal name="N$2">
@@
 <contactref element="C9" pad="2"/>
 <contactref element="OP1" pad="2"/>
-<wire x1="5.9826" y1="2.7178" x2="9.8416" y2="-6.9088" width="0" layer="19" extent="1-1"/>
-<wire x1="7.9502" y1="19.0154" x2="5.9826" y2="2.7178" width="0" layer="19" extent="1-1"/>
+<wire x1="5.9826" y1="2.7178" x2="7.9502" y2="19.0154" width="0" layer="19" extent="1-1"/>
+<wire x1="9.8416" y1="-6.9088" x2="5.9826" y2="2.7178" width="0" layer="19" extent="1-1"/>
 </signal>
 <signal name="N$4">
@@
 <contactref element="R11" pad="2"/>
 <contactref element="OP1" pad="3"/>
-<wire x1="13.374" y1="-8.1534" x2="11.9498" y2="-9.525" width="0" layer="19" extent="1-1"/>
-<wire x1="9.2202" y1="19.0154" x2="13.374" y2="-8.1534" width="0" layer="19" extent="1-1"/>
+<wire x1="13.374" y1="-8.1534" x2="9.2202" y2="19.0154" width="0" layer="19" extent="1-1"/>
+<wire x1="11.9498" y1="-9.525" x2="13.374" y2="-8.1534" width="0" layer="19" extent="1-1"/>
 </signal>
 <signal name="N$5">
@@
 <contactref element="OP1" pad="1"/>
 <contactref element="OP2" pad="5"/>
-<wire x1="7.6826" y1="2.7178" x2="15.074" y2="-8.1534" width="0" layer="19" extent="1-1"/>
-<wire x1="21.4884" y1="22.9962" x2="7.6826" y2="2.7178" width="0" layer="19" extent="1-1"/>
 <wire x1="6.6802" y1="19.0154" x2="21.4884" y2="22.9962" width="0" layer="19" extent="1-1"/>
+<wire x1="7.6826" y1="2.7178" x2="6.6802" y2="19.0154" width="0" layer="19" extent="1-1"/>
+<wire x1="15.074" y1="-8.1534" x2="7.6826" y2="2.7178" width="0" layer="19" extent="1-1"/>
 </signal>
 <signal name="N$6">
@@
 <contactref element="OP2" pad="6"/>
 <contactref element="OP2" pad="7"/>
-<wire x1="18.9484" y1="22.9962" x2="18.1746" y2="-8.6614" width="0" layer="19" extent="1-1"/>
-<wire x1="20.2184" y1="22.9962" x2="18.9484" y2="22.9962" width="0" layer="19" extent="1-1"/>
+<wire x1="18.9484" y1="22.9962" x2="20.2184" y2="22.9962" width="0" layer="19" extent="1-1"/>
+<wire x1="18.1746" y1="-8.6614" x2="18.9484" y2="22.9962" width="0" layer="19" extent="1-1"/>
 </signal>
 <signal name="N$7">
 <contactref element="Q1" pad="1"/>
 <contactref element="R12" pad="2"/>
-<wire x1="11.115" y1="2.175" x2="19.8746" y2="-8.6614" width="0" layer="19" extent="1-1"/>
+<wire x1="19.8746" y1="-8.6614" x2="11.115" y2="2.175" width="0" layer="19" extent="1-1"/>
 </signal>
 <signal name="N$11">
@@
 <wire x1="3.81" y1="6.5278" x2="3.7338" y2="-0.1016" width="0" layer="19" extent="1-1"/>
 <wire x1="3.937" y1="13.3604" x2="3.81" y2="6.5278" width="0" layer="19" extent="1-1"/>
-<wire x1="12.065" y1="4.275" x2="3.937" y2="13.3604" width="0" layer="19" extent="1-1"/>
+<wire x1="12.065" y1="4.275" x2="3.81" y2="6.5278" width="0" layer="19" extent="1-1"/>
 </signal>
 </signals>
