File: Hardware/BlinkyCircuit.brd (EAGLE design)
At the start: 170.5 x 81 mm, 22 parts

Commit message: March 27 2021 edits
Parts:
- added J1: (no value), LinnesLab-Connectors:1X02
- moved LED5 233.4 mm to (223.0, 75.9)
- moved LED6 229.2 mm to (215.0, 75.8)
- moved LED7 228.1 mm to (206.3, 75.8)
- moved LED21 224.8 mm to (197.7, 76.7)
- moved LED1 222.6 mm to (188.3, 77.8)
- moved LED8 221.3 mm to (179.2, 78.7)
- moved LED9 219.1 mm to (170.3, 80.6)
- moved LED3 179.9 mm to (153.5, 104.3)
- moved LED2 174.1 mm to (162.3, 82.7)
- moved LED4 159.3 mm to (122.7, 104.4)
- moved R11 133.6 mm to (98.5, 91.5), flipped to the bottom, turned to 270 degrees
- moved C9 132.9 mm to (89.7, 98.7), flipped to the bottom, turned to 270 degrees
- moved R12 131.7 mm to (101.9, 93.7), flipped to the bottom, turned to 270 degrees
- moved R8 131.2 mm to (99.3, 95.8), flipped to the bottom, turned to 270 degrees
- moved Q1 130.8 mm to (110.0, 89.9), flipped to the bottom, turned to 90 degrees
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Connections:
- net GND: now also J1.2
- net V_BATT: now also J1.1
Routing:
- net N$2: track 0.00 -> 81.8 mm
- net N$11: track 0.00 -> 61.3 mm
- net N$5: track 0.00 -> 16.9 mm
- net N$3: track 0.00 -> 16.2 mm
- net GND: track 0.00 -> 9.96 mm
- net N$7: track 0.00 -> 8.67 mm
- net V_BATT: track 0.00 -> 8.36 mm
- net N$1: track 0.00 -> 5.48 mm
- net N$6: track 0.00 -> 4.08 mm
- net N$4: track 0.00 -> 2.64 mm
Other:
- board size 170.5 x 81 mm -> 170.5 x 83.7 mm

Commit message: March 27 2021 board edits
Parts:
- moved C7 15.5 mm to (85.3, 94.9)
- moved Q1 15.0 mm to (100.7, 101.7), turned to 0 degrees
- moved C8 9.27 mm to (87.3, 94.9)
- moved R10 7.84 mm to (99.6, 94.2), turned to 90 degrees
- moved R9 6.75 mm to (88.8, 88.8), turned to 0 degrees
- moved R11 5.36 mm to (93.3, 89.9), turned to 180 degrees
- moved R12 2.48 mm to (102.2, 96.1), turned to 0 degrees
- moved OP2 2.37 mm to (107.0, 96.8)
- moved R8 1.86 mm to (97.5, 95.2), turned to 90 degrees
- moved C9 1.26 mm to (90.5, 97.7), turned to 180 degrees
- moved R7 0.26 mm to (87.0, 91.4), turned to 90 degrees
Routing:
- net N$2: track 81.8 -> 2.47 mm
- net N$11: track 61.3 -> 0.00 mm
- net GND: track 9.96 -> 0.00 mm
- net V_BATT: track 8.36 -> 0.27 mm
- net N$4: track 2.64 -> 10.4 mm
- net N$5: track 16.9 -> 9.76 mm
- net N$6: track 4.08 -> 0.00 mm
- net N$7: track 8.67 -> 4.71 mm
- net N$3: track 16.2 -> 13.4 mm
